File: pcb/h_bridge_controller.sch (KiCad schematic (older format))
At the start: 58 parts, among them P1 PWR_JACK_2.5x5.5, P10 HEADER_02X08_SMD, P11 HEADER_02X08_SMD, P2 HEADER_01X03_SMD_RA, P3 HEADER_01X03_SMD_RA, P4 HEADER_01X03_SMD_RA, P5 HEADER_01X03_SMD_RA, P6 HEADER_01X02_SMD_RA, P7 BNC_DOUBLE_RA, P8 HEADER_02X08_SMD, P9 HEADER_02X08_SMD, SW1 SPST_SLIDE_AS, U1 TLE7230R, U2 TLE7230R, U3 TLE7230R, U4 TLE7230R

Commit message: Progress towards pcb v1.0.
Parts:
- removed C4, C6, C7: 0.1uF, h_bridge_controller:SM1210, symbol 0.1uF
- removed D1, D10, D11, D12, D13, D14, D15, D16, D17, D18, D19, D2, D20, D21, D22, D23, D24, D25, D26, D27, D28, D29, D3, D30, D31, D32, D33, D4, D5, D6, D7, D8, D9: LED_24V, h_bridge_controller:LED_555-3XXX, symbol LED_24V
- removed P10, P11, P8, P9: HEADER_02X08_SMD, h_bridge_controller:HEADER_02x08_SMD, symbol HEADER_02X08_SMD
- removed U1, U2, U3, U4: TLE7230R, h_bridge_controller:PG-DSO-36, symbol TLE7230R
- added C4: 10uF, h_bridge_controller:SM1210, symbol 10uF
- added D1, D2, D3, D4, D5, D6, D7, D8: diode_schottky_40V_1A, h_bridge_controller:DO-214AC(SMA), symbol diode_schottky_40V_1A
- added L1, L2, L3, L4, L5: LED_24V, h_bridge_controller:LED_555-3XXX, symbol LED_24V
- added P8: SPR_TERM_0.1_01X04, h_bridge_controller:SPRING_TERM_BLK_0.1_4, symbol SPR_TERM_0.1_01X04
- added U1: L298, h_bridge_controller:POWERSO20, symbol L298
Connections:
- net labels added: DIR0A, DIR0B, DIR1A, DIR1B, PWM0, PWM1, SENA, SENB
- net labels removed: CS, MISO, MOSI, OUT10, OUT11, OUT12, OUT13, OUT14, OUT15, OUT16, OUT17, OUT18, OUT19, OUT20, OUT21, OUT22, OUT23, OUT24, OUT25, OUT26, OUT27, OUT28, OUT29, OUT30, OUT31, OUT4, OUT5, OUT6, OUT7, OUT8, OUT9, RESET, SCK, SO1, SO2, SO3
- wire segments 313 -> 122
- no-connect marks 73 -> 70

Commit message: Use relay_controller as pcb base.
Parts:
- removed C4: 10uF, h_bridge_controller:SM1210, symbol 10uF
- removed C5: 0.1uF, h_bridge_controller:SM1210, symbol 0.1uF
- removed D1, D2, D3, D4, D5, D6, D7, D8: diode_schottky_40V_1A, h_bridge_controller:DO-214AC(SMA), symbol diode_schottky_40V_1A
- removed L2, L3, L4, L5: LED_24V, h_bridge_controller:LED_555-3XXX, symbol LED_24V
- removed P8: SPR_TERM_0.1_01X04, h_bridge_controller:SPRING_TERM_BLK_0.1_4, symbol SPR_TERM_0.1_01X04
- removed U1: L298, h_bridge_controller:POWERSO20, symbol L298
- added L2, L3, L4, L5, L6, L7, L8, L9: LED_5V_GRN, relay_controller:LED_555-3XXX, symbol LED_5V_GRN
- added R1: 5.11k, relay_controller:SM1210, symbol 5.11k
- added R10, R3, R4, R5, R6, R7, R8, R9: 150, relay_controller:SM1210, symbol 150
- added R2: 1k, relay_controller:SM1210, symbol 1k
- added T1, T2, T3, T4, T5, T6, T7, T8: TERM_BLK_ANG_2_PIN, relay_controller:TERM_BLK_ANG_2_PIN, symbol TERM_BLK_ANG_2_PIN
- added U1, U2, U3, U4, U5, U6, U7, U8: SSR_DC_6PIN, relay_controller:ASSR-1611, symbol SSR_DC_6PIN
- ARDUINO1: footprint h_bridge_controller:ARDUINO_MEGA_SHIELD -> relay_controller:ARDUINO_MEGA_SHIELD
- C1, C2, C3: footprint h_bridge_controller:SM1210 -> relay_controller:SM1210
- L1: footprint h_bridge_controller:LED_555-3XXX -> relay_controller:LED_555-3XXX
- P1: footprint h_bridge_controller:DCJACK_2PIN_HIGHCURRENT -> relay_controller:DCJACK_2PIN_HIGHCURRENT
- P2, P3, P4, P5: footprint h_bridge_controller:Header_3_Pin_SMD_RA -> relay_controller:Header_3_Pin_SMD_RA
- P6: footprint h_bridge_controller:Header_2_Pin_SMD_RA -> relay_controller:Header_2_Pin_SMD_RA
- P7: footprint h_bridge_controller:BNC_DOUBLE -> relay_controller:BNC_DOUBLE
- REG1: footprint h_bridge_controller:DC_DC_CONV_R78C -> relay_controller:DC_DC_CONV_R78C
- SW1: footprint h_bridge_controller:SPST_SLIDE_AS -> relay_controller:SPST_SLIDE_AS
Connections:
- net labels added: LED_0, LED_1, LED_2, LED_3, LED_4, LED_5, LED_6, LED_7, LED_PWR_IN, OUT_0+, OUT_0-, OUT_1+, OUT_1-, OUT_2+, OUT_2-, OUT_3+, OUT_3-, OUT_4+, OUT_4-, OUT_5+, OUT_5-, OUT_6+, OUT_6-, OUT_7+, OUT_7-, RELAY_0, RELAY_1, RELAY_2, RELAY_3, RELAY_4, RELAY_5, RELAY_6, RELAY_7
- net labels removed: DIR0A, DIR0B, DIR1A, DIR1B, OUT0, OUT1, OUT2, OUT3, PWM0, PWM1, SENA, SENB
- wire segments 122 -> 187
- no-connect marks 70 -> 53
Other:
- moved on the sheet: C1, C2, C3, P1, P2, P3, P4, P5, P6, P7, REG1, SW1

Commit message: relay_controller -> h_bridge_controller.
Parts:
- ARDUINO1: footprint relay_controller:ARDUINO_MEGA_SHIELD -> h_bridge_controller:ARDUINO_MEGA_SHIELD
- C1, C2, C3, R1, R10, R2, R3, R4, R5, R6, R7, R8, R9: footprint relay_controller:SM1210 -> h_bridge_controller:SM1210
- L1, L2, L3, L4, L5, L6, L7, L8, L9: footprint relay_controller:LED_555-3XXX -> h_bridge_controller:LED_555-3XXX
- P1: footprint relay_controller:DCJACK_2PIN_HIGHCURRENT -> h_bridge_controller:DCJACK_2PIN_HIGHCURRENT
- P2, P3, P4, P5: footprint relay_controller:Header_3_Pin_SMD_RA -> h_bridge_controller:Header_3_Pin_SMD_RA
- P6: footprint relay_controller:Header_2_Pin_SMD_RA -> h_bridge_controller:Header_2_Pin_SMD_RA
- P7: footprint relay_controller:BNC_DOUBLE -> h_bridge_controller:BNC_DOUBLE
- REG1: footprint relay_controller:DC_DC_CONV_R78C -> h_bridge_controller:DC_DC_CONV_R78C
- SW1: footprint relay_controller:SPST_SLIDE_AS -> h_bridge_controller:SPST_SLIDE_AS
- T1, T2, T3, T4, T5, T6, T7, T8: footprint relay_controller:TERM_BLK_ANG_2_PIN -> h_bridge_controller:TERM_BLK_ANG_2_PIN
- U1, U2, U3, U4, U5, U6, U7, U8: footprint relay_controller:ASSR-1611 -> h_bridge_controller:ASSR-1611

Commit message: Progress towards pcb1.0.
Parts:
- removed L2, L3, L4, L5, L6, L7, L8, L9: LED_5V_GRN, h_bridge_controller:LED_555-3XXX, symbol LED_5V_GRN
- removed R10, R3, R4, R5, R6, R7, R8, R9: 150, h_bridge_controller:SM1210, symbol 150
- removed T3, T4, T5, T6, T7, T8: TERM_BLK_ANG_2_PIN, h_bridge_controller:TERM_BLK_ANG_2_PIN, symbol TERM_BLK_ANG_2_PIN
- removed U1, U2, U3, U4, U5, U6, U7, U8: SSR_DC_6PIN, h_bridge_controller:ASSR-1611, symbol SSR_DC_6PIN
- added C4: 10uF, h_bridge_controller:SM1210, symbol 10uF
- added C5: 0.1uF, h_bridge_controller:SM1210, symbol 0.1uF
- added D1, D2, D3, D4, D5, D6, D7, D8: diode_schottky_40V_1A, h_bridge_controller:DO-214AC(SMA), symbol diode_schottky_40V_1A
- added L2, L3, L4, L5: LED_24V, h_bridge_controller:LED_555-3XXX, symbol LED_24V
- added U1: L298, h_bridge_controller:POWERSO20, symbol L298
Connections:
- net +5V: now also C5.1, U1.12 (Vss)
- net GND: now also C4.2, C5.2, D2.2 (A), D4.2 (A), D6.2 (A), D8.2 (A), U1.1 (GND), U1.10 (GND), U1.11 (GND), U1.20 (GND)
- net LED_PWR: now also L2.1 (A), L3.1 (A), L4.1 (A), L5.1 (A)
- net OUT_0+: now also D1.2 (A), D2.1 (K), L2.2 (K), U1.4 (OUT1)
- net OUT_0-: now also D3.2 (A), D4.1 (K), L3.2 (K), U1.5 (OUT2)
- net OUT_1+: now also D5.2 (A), D6.1 (K), L4.2 (K), U1.16 (OUT3)
- net OUT_1-: now also D7.2 (A), D8.1 (K), L5.2 (K), U1.17 (OUT4)
- net VAA: now also C4.1, D1.1 (K), D3.1 (K), D5.1 (K), D7.1 (K), U1.6 (Vs)
- net LED_0: no longer names the net of ARDUINO1.22 (D22/AD0/PA0)
- net LED_1: no longer names the net of ARDUINO1.23 (D23/AD1/PA1)
- net LED_2: no longer names the net of ARDUINO1.24 (D24/AD2/PA2)
- net LED_3: no longer names the net of ARDUINO1.25 (D25/AD3/PA3)
- net LED_4: no longer names the net of ARDUINO1.26 (D26/AD4/PA4)
- net LED_5: no longer names the net of ARDUINO1.27 (D27/AD5/PA5)
- net LED_6: no longer names the net of ARDUINO1.28 (D28/AD6/PA6)
- net LED_7: no longer names the net of ARDUINO1.29 (D29/AD7/PA7)
- net RELAY_0: no longer names the net of ARDUINO1.38 (D38/T0/PD7)
- net RELAY_1: no longer names the net of ARDUINO1.39 (D39/ALE/PG2)
- net RELAY_2: no longer names the net of ARDUINO1.40 (D40/RD/PG1)
- net RELAY_3: no longer names the net of ARDUINO1.41 (D41/WR/PG0)
- net RELAY_4: no longer names the net of ARDUINO1.42 (D42/PL7)
- net RELAY_5: no longer names the net of ARDUINO1.43 (D43/PL6)
- net RELAY_6: no longer names the net of ARDUINO1.44 (D44/PWM/OC5C/PL5)
- net RELAY_7: no longer names the net of ARDUINO1.45 (D45/PWM/OC5B/PL4)
- new net DIR_0A: U1.7 (IN1)
- new net DIR_0B: U1.9 (IN2)
- new net DIR_1A: U1.13 (IN3)
- new net DIR_1B: U1.15 (IN4)
- new net PWM_0: U1.8 (ENA)
- new net PWM_1: U1.14 (ENB)
- new net SENSE_0: U1.2 (SENA)
- new net SENSE_1: U1.19 (SENB)
- no-connect marks 53 -> 69

Commit message: Progress towards pcb1.0.
Parts:
- removed C4: 10uF, h_bridge_controller:SM1210, symbol 10uF
- removed R1: 5.11k, h_bridge_controller:SM1210, symbol 5.11k
- removed R2: 1k, h_bridge_controller:SM1210, symbol 1k
- added C4, C7, C8: 0.1uF, h_bridge_controller:SM1210, symbol 0.1uF
- added C6, C9: 47uF, h_bridge_controller:SM2917_POL, symbol 47uF_2917_POL
- added D10, D11, D12, D13, D14, D15, D16, D9: diode_schottky_40V_1A, h_bridge_controller:DO-214AC(SMA), symbol diode_schottky_40V_1A
- added L6, L7, L8, L9: LED_24V, h_bridge_controller:LED_555-3XXX, symbol LED_24V
- added P10, P8, P9: HEADER_01X05_SMD_SHR, h_bridge_controller:Header_Shrouded_5_Pin_SMD, symbol HEADER_01X05_SMD_SHR
- added R1, R2, R3, R4: 0.5_2010, h_bridge_controller:SM2010, symbol 0.5_2010
- added R7, R8, R9: 180, h_bridge_controller:SM1210, symbol 180
- added T3, T4: TERM_BLK_ANG_2_PIN, h_bridge_controller:TERM_BLK_ANG_2_PIN, symbol TERM_BLK_ANG_2_PIN
- added U2: L298, h_bridge_controller:POWERSO20, symbol L298
Connections:
- net +5V: now also C8.1, P10.3 (P3), P8.3 (P3), P9.3 (P3), R7.2, R8.2, R9.2, U2.12 (Vss)
- net DIR_0A: now also ARDUINO1.22 (D22/AD0/PA0)
- net DIR_0B: now also ARDUINO1.23 (D23/AD1/PA1)
- net DIR_1A: now also ARDUINO1.24 (D24/AD2/PA2)
- net DIR_1B: now also ARDUINO1.25 (D25/AD3/PA3)
- net GND: now also C4.2, C6.2, C7.2, C8.2, C9.2, D10.2 (A), D12.2 (A), D14.2 (A), D16.2 (A), P10.2 (P2), P10.5 (P5), P8.2 (P2), P8.5 (P5), P9.2 (P2), P9.5 (P5), R1.2, R2.2, R3.2, R4.2, U2.1 (GND), U2.10 (GND), U2.11 (GND), U2.20 (GND)
- net LED_PWR: now also L6.1 (A), L7.1 (A), L8.1 (A), L9.1 (A)
- net PWM_0: now also ARDUINO1.8 (D8/PWM/OC4C/PH5)
- net PWM_1: now also ARDUINO1.9 (D9/PWM/OC2B/PH6)
- net SENSE_0: now also ARDUINO1.A0 (A0/PF0), R1.1
- net SENSE_1: now also ARDUINO1.A1 (A1/PF1), R2.1
- net VAA: now also C4.1, C6.1, C7.1, C9.1, D11.1 (K), D13.1 (K), D15.1 (K), D9.1 (K), U2.6 (Vs)
- net PWM_2: now reaches ARDUINO1.10 (D10/PWM/OC2A/PCINT4/PB4)
- net PWM_2: now also U2.8 (ENA)
- net PWM_3: now reaches ARDUINO1.11 (D11/PWM/OC1A/PCINT5/PB5)
- net PWM_3: now also U2.14 (ENB)
- net SW_2: now reaches ARDUINO1.2 (D2/PWM/OC3B/INT4/PE4)
- net SW_2: now also P10.4 (P4)
- net SW_1: now reaches ARDUINO1.20 (D20/SDA/INT1/PD1)
- net SW_1: now also P9.4 (P4)
- net SW_0: now reaches ARDUINO1.21 (D21/SCL/INT0/PD0)
- net SW_0: now also P8.4 (P4)
- net DIR_2A: now reaches ARDUINO1.26 (D26/AD4/PA4)
- net DIR_2A: now also U2.7 (IN1)
- net DIR_2B: now reaches ARDUINO1.27 (D27/AD5/PA5)
- net DIR_2B: now also U2.9 (IN2)
- net DIR_3A: now reaches ARDUINO1.28 (D28/AD6/PA6)
- net DIR_3A: now also U2.13 (IN3)
- net DIR_3B: now reaches ARDUINO1.29 (D29/AD7/PA7)
- net DIR_3B: now also U2.15 (IN4)
- net SENSE_2: now reaches ARDUINO1.A2 (A2/PF2)
- net SENSE_2: now also R3.1, U2.2 (SENA)
- net SENSE_3: now reaches ARDUINO1.A3 (A3/PF3)
- net SENSE_3: now also R4.1, U2.19 (SENB)
- net LED_PWR_IN: no longer names the net of ARDUINO1.33 (D33/A12/PC4)
- new net: P8.1 (P1), R7.1
- new net: P9.1 (P1), R8.1
- new net: P10.1 (P1), R9.1
- new net OUT_2+: D10.1 (K), D9.2 (A), L6.2 (K), T3.1 (P1), U2.4 (OUT1)
- new net OUT_2-: D11.2 (A), D12.1 (K), L7.2 (K), T3.2 (P2), U2.5 (OUT2)
- new net OUT_3+: D13.2 (A), D14.1 (K), L8.2 (K), T4.1 (P1), U2.16 (OUT3)
- new net OUT_3-: D15.2 (A), D16.1 (K), L9.2 (K), T4.2 (P2), U2.17 (OUT4)
- no-connect marks 69 -> 51
Other:
- moved on the sheet: C5, D1, D2, D3, D4, D5, D6, D7, D8, L2, L3, L4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

Commit message: More progress towards pcb1.0.
Parts:
- R1, R2, R3, R4: value 0.5_2010 -> 0.5
Connections:
- net GND: now also SW1.1; no longer L1.2 (K)
- net OUT_0+: now also L2.1 (A); no longer L2.2 (K)
- net OUT_0-: now also L3.1 (A); no longer L3.2 (K)
- net OUT_1+: now also L4.1 (A); no longer L4.2 (K)
- net OUT_1-: now also L5.1 (A); no longer L5.2 (K)
- net OUT_2+: now also L6.1 (A); no longer L6.2 (K)
- net OUT_2-: now also L7.1 (A); no longer L7.2 (K)
- net OUT_3+: now also L8.1 (A); no longer L8.2 (K)
- net OUT_3-: now also L9.1 (A); no longer L9.2 (K)
- net VAA: now also L1.1 (A); no longer SW1.1
- removed net LED_PWR: L1.1 (A), L2.1 (A), L3.1 (A), L4.1 (A), L5.1 (A), L6.1 (A), L7.1 (A), L8.1 (A), L9.1 (A), SW1.3
- net PWM_0 renamed ENABLE_0
- net PWM_1 renamed ENABLE_1
- net PWM_2 renamed ENABLE_2
- net PWM_3 renamed ENABLE_3
- new net LED_GND: L1.2 (K), L2.2 (K), L3.2 (K), L4.2 (K), L5.2 (K), L6.2 (K), L7.2 (K), L8.2 (K), L9.2 (K), SW1.3

Commit message: Finished pcb1.0.
Connections:
- net DIR_0A: now also ARDUINO1.30 (D30/A15/PC7); no longer ARDUINO1.22 (D22/AD0/PA0)
- net DIR_0B: now also ARDUINO1.31 (D31/A14/PC6); no longer ARDUINO1.23 (D23/AD1/PA1)
- net DIR_1A: now also ARDUINO1.32 (D32/A13/PC5); no longer ARDUINO1.24 (D24/AD2/PA2)
- net DIR_1B: now also ARDUINO1.33 (D33/A12/PC4); no longer ARDUINO1.25 (D25/AD3/PA3)
- net DIR_2A: now also ARDUINO1.34 (D34/A11/PC3); no longer ARDUINO1.26 (D26/AD4/PA4)
- net DIR_2B: now also ARDUINO1.35 (D35/A10/PC2); no longer ARDUINO1.27 (D27/AD5/PA5)
- net DIR_3A: now also ARDUINO1.36 (D36/A9/PC1); no longer ARDUINO1.28 (D28/AD6/PA6)
- net DIR_3B: now also ARDUINO1.37 (D37/A8/PC0); no longer ARDUINO1.29 (D29/AD7/PA7)
Changed lines of the file:
@@
 	700  1250 700  1600
 Wire Wire Line
-	700  1600 850  1600
-Wire Wire Line
-	850  1600 1350 1600
+	700  1600 1350 1600
 Wire Wire Line
 	850  1250 850  1600
@@
 	1350 1700 850  1700
 Wire Wire Line
-	850  1700 850  1800
-Wire Wire Line
-	850  1800 850  1850
+	850  1700 850  1850
 Wire Wire Line
 	1350 1800 850  1800
@@
 NoConn ~ 3550 2000
 NoConn ~ 3550 3850
-NoConn ~ 3550 4850
-NoConn ~ 3550 4950
 $Comp
 L GND #PWR04
@@
 $EndComp
 Wire Wire Line
-	800  7550 950  7550
-Wire Wire Line
-	950  7550 1050 7550
+	800  7550 1050 7550
 Wire Wire Line
 	800  7550 800  7450
@@
 Connection ~ 950  7550
 Wire Wire Line
-	600  7650 950  7650
-Wire Wire Line
-	950  7650 1050 7650
+	600  7650 1050 7650
 Wire Wire Line
 	600  7650 600  7550
@@
 	5300 7600 5400 7600
 Wire Wire Line
-	5400 7600 5400 7700
-Wire Wire Line
-	5400 7700 5400 7850
+	5400 7600 5400 7850
 Wire Wire Line
 	5300 7700 5400 7700
@@
 	4150 3750 4150 3700
 Wire Wire Line
-	3550 3750 3800 3750
-Wire Wire Line
-	3800 3750 4150 3750
+	3550 3750 4150 3750
 Wire Wire Line
 	3800 3700 3800 3750
@@
 Wire Wire Line
 	3550 2300 3750 2300
-NoConn ~ 3550 5050
 Wire Wire Line
 	3550 2600 3750 2600
@@
 $EndComp
 Wire Wire Line
-	2700 7250 2700 7300
-Wire Wire Line
-	2700 7300 2700 7350
-Wire Wire Line
-	2700 7300 2950 7300
-Wire Wire Line
-	2950 7300 3150 7300
+	2700 7250 2700 7350
+Wire Wire Line
+	2700 7300 3150 7300
 Connection ~ 2700 7300
 Wire Wire Line
 	2700 7750 2700 7800
 Wire Wire Line
-	2700 7800 2950 7800
-Wire Wire Line
-	2950 7800 3550 7800
-Wire Wire Line
-	3550 7800 4050 7800
+	2700 7800 4050 7800
 Wire Wire Line
 	4050 7800 4050 7750
 Wire Wire Line
-	3550 7650 3550 7800
-Wire Wire Line
-	3550 7800 3550 7850
+	3550 7650 3550 7850
 Connection ~ 3550 7800
 Wire Wire Line
@@
 Connection ~ 2950 7800
 Wire Wire Line
-	3950 7300 4050 7300
-Wire Wire Line
-	4050 7300 4150 7300
+	3950 7300 4150 7300
 Wire Wire Line
 	4050 7350 4050 7300
@@
 	5450 1850 5450 1900
 Wire Wire Line
-	5450 1900 5550 1900
-Wire Wire Line
-	5550 1900 5600 1900
-Wire Wire Line
-	5600 1900 5650 1900
-Wire Wire Line
-	5650 1900 5750 1900
+	5450 1900 5750 1900
 Wire Wire Line
 	5750 1900 5750 1850
@@
 	7700 750  7700 800
 Wire Wire Line
-	7700 1000 7700 1050
-Wire Wire Line
-	7700 1050 7700 1100
+	7700 1000 7700 1100
 Wire Wire Line
 	7700 1300 7700 1350
@@
 	8200 750  8200 800
 Wire Wire Line
-	8200 1000 8200 1050
-Wire Wire Line
-	8200 1050 8200 1100
+	8200 1000 8200 1100
 Wire Wire Line
 	8200 1300 8200 1350
@@
 	8700 750  8700 800
 Wire Wire Line
-	8700 1000 8700 1050
-Wire Wire Line
-	8700 1050 8700 1100
+	8700 1000 8700 1100
 Wire Wire Line
 	8700 1300 8700 1350
@@
 	9200 750  9200 800
 Wire Wire Line
-	9200 1000 9200 1050
-Wire Wire Line
-	9200 1050 9200 1100
+	9200 1000 9200 1100
 Wire Wire Line
 	9200 1300 9200 1350
@@
 Text Label 3750 1600 0    60   ~ 0
 ENABLE_1
-Text Label 3750 4000 0    60   ~ 0
+Text Label 3750 4850 0    60   ~ 0
 DIR_0A
-Text Label 3750 4100 0    60   ~ 0
+Text Label 3750 4950 0    60   ~ 0
 DIR_0B
-Text Label 3750 4200 0    60   ~ 0
+Text Label 3750 5050 0    60   ~ 0
 DIR_1A
-Text Label 3750 4300 0    60   ~ 0
+Text Label 3750 5150 0    60   ~ 0
 DIR_1B
 $Comp
@@
 	6450 6500 6350 6500
 Wire Wire Line
-	6350 6200 6350 6500
-Wire Wire Line
-	6350 6500 6350 6600
+	6350 6200 6350 6600
 Wire Wire Line
 	6450 6200 6350 6200
@@
 $EndComp
 Wire Wire Line
-	5800 6000 5800 6100
-Wire Wire Line
-	5800 6100 5800 6300
+	5800 6000 5800 6300
 Wire Wire Line
 	5800 6100 5900 6100
@@
 	7550 6500 7450 6500
 Wire Wire Line
-	7450 6200 7450 6500
-Wire Wire Line
-	7450 6500 7450 6600
+	7450 6200 7450 6600
 Wire Wire Line
 	7550 6200 7450 6200
@@
 $EndComp
 Wire Wire Line
-	6900 6000 6900 6100
-Wire Wire Line
-	6900 6100 6900 6300
+	6900 6000 6900 6300
 Wire Wire Line
 	6900 6100 7000 6100
@@
 	8650 6500 8550 6500
 Wire Wire Line
-	8550 6200 8550 6500
-Wire Wire Line
-	8550 6500 8550 6600
+	8550 6200 8550 6600
 Wire Wire Line
 	8650 6200 8550 6200
@@
 $EndComp
 Wire Wire Line
-	8000 6000 8000 6100
-Wire Wire Line
-	8000 6100 8000 6300
+	8000 6000 8000 6300
 Wire Wire Line
 	8000 6100 8100 6100
@@
 Wire Wire Line
 	3550 1400 3750 1400
-NoConn ~ 3550 5250
-NoConn ~ 3550 5350
-NoConn ~ 3550 5450
-NoConn ~ 3550 5550
-Wire Wire Line
-	3550 4000 3750 4000
-Wire Wire Line
-	3550 4100 3750 4100
-Wire Wire Line
-	3550 4200 3750 4200
-Wire Wire Line
-	3550 4300 3750 4300
 $Comp
 L L298 U2
@@
 	5450 4600 5450 4650
 Wire Wire Line
-	5450 4650 5550 4650
-Wire Wire Line
-	5550 4650 5600 4650
-Wire Wire Line
-	5600 4650 5650 4650
-Wire Wire Line
-	5650 4650 5750 4650
+	5450 4650 5750 4650
 Wire Wire Line
 	5750 4650 5750 4600
@@
 	7700 3500 7700 3550
 Wire Wire Line
-	7700 3750 7700 3800
-Wire Wire Line
-	7700 3800 7700 3850
+	7700 3750 7700 3850
 Wire Wire Line
 	7700 4050 7700 4100
@@
 	8200 3500 8200 3550
 Wire Wire Line
-	8200 3750 8200 3800
-Wire Wire Line
-	8200 3800 8200 3850
+	8200 3750 8200 3850
 Wire Wire Line
 	8200 4050 8200 4100
@@
 	8700 3500 8700 3550
 Wire Wire Line
-	8700 3750 8700 3800
-Wire Wire Line
-	8700 3800 8700 3850
+	8700 3750 8700 3850
 Wire Wire Line
 	8700 4050 8700 4100
@@
 	9200 3500 9200 3550
 Wire Wire Line
-	9200 3750 9200 3800
-Wire Wire Line
-	9200 3800 9200 3850
+	9200 3750 9200 3850
 Wire Wire Line
 	9200 4050 9200 4100
@@
 	1    0    0    -1
 $EndComp
-Text Label 3750 4400 0    60   ~ 0
+Text Label 3750 5250 0    60   ~ 0
 DIR_2A
-Text Label 3750 4500 0    60   ~ 0
+Text Label 3750 5350 0    60   ~ 0
 DIR_2B
-Text Label 3750 4600 0    60   ~ 0
+Text Label 3750 5450 0    60   ~ 0
 DIR_3A
-Text Label 3750 4700 0    60   ~ 0
+Text Label 3750 5550 0    60   ~ 0
 DIR_3B
-Wire Wire Line
-	3550 4400 3750 4400
-Wire Wire Line
-	3550 4500 3750 4500
-Wire Wire Line
-	3550 4600 3750 4600
-Wire Wire Line
-	3550 4700 3750 4700
 Text Label 3750 1500 0    60   ~ 0
 ENABLE_2
@@
 Text Label 900  2400 0    60   ~ 0
 SENSE_3
-NoConn ~ 3550 5150
 $Comp
 L HEADER_01X05_SMD_SHR P8
@@
 	7700 2200 7700 2250
 Wire Wire Line
-	7700 2250 8200 2250
-Wire Wire Line
-	8200 2250 8450 2250
-Wire Wire Line
-	8450 2250 8700 2250
-Wire Wire Line
-	8700 2250 9200 2250
+	7700 2250 9200 2250
 Wire Wire Line
 	8700 2200 8700 2250
@@
 	7700 4950 7700 5000
 Wire Wire Line
-	7700 5000 8200 5000
-Wire Wire Line
-	8200 5000 8450 5000
-Wire Wire Line
-	8450 5000 8700 5000
-Wire Wire Line
-	8700 5000 9200 5000
+	7700 5000 9200 5000
 Wire Wire Line
 	9200 5000 9200 4950
@@
 	8450 5100 8450 5000
 Connection ~ 8450 5000
+Wire Wire Line
+	3550 4850 3750 4850
+Wire Wire Line
+	3550 4950 3750 4950
+Wire Wire Line
+	3550 5050 3750 5050
+Wire Wire Line
+	3550 5150 3750 5150
+Wire Wire Line
+	3550 5250 3750 5250
+Wire Wire Line
+	3550 5350 3750 5350
+Wire Wire Line
+	3550 5450 3750 5450
+Wire Wire Line
+	3550 5550 3750 5550
+NoConn ~ 3550 4700
+NoConn ~ 3550 4600
+NoConn ~ 3550 4500
+NoConn ~ 3550 4400
+NoConn ~ 3550 4300
+NoConn ~ 3550 4200
+NoConn ~ 3550 4100
+NoConn ~ 3550 4000
 $EndSCHEMATC
